Commit message: Make package more generic to work with multiple robots

File: lwr_robot_examples/kuka-lwr-single/lwr_robot/single_lwr_robot/robot/single_lwr_robot.urdf.xacro (robot description, xacro)
@@ -1,9 +1,15 @@
 <?xml version="1.0"?>
 <robot xmlns:xacro="http://www.ros.org/wiki/xacro" name="single_lwr_robot">
-  <!-- Include all models -->
+  <xacro:arg name="robot_name" default="lwr"/>
+  <xacro:arg name="robot_world" default="world"/>
+  <xacro:arg name="robot_origin.x" default="0"/>
+  <xacro:arg name="robot_origin.y" default="0"/>
+  <xacro:arg name="robot_origin.z" default="0"/>
+  <xacro:arg name="robot_origin.ax" default="0"/>
+  <xacro:arg name="robot_origin.ay" default="0"/>
+  <xacro:arg name="robot_origin.az" default="0"/>  <!-- Include all models -->
   <xacro:include filename="$(find lwr_description)/model/kuka_lwr.urdf.xacro"/>
-  <!-- using the models -->
-  <xacro:kuka_lwr name="lwr">
-    <origin xyz="0 0 0" rpy="0 0 0"/>
+  <xacro:kuka_lwr base_link="$(arg robot_world)" name="$(arg robot_name)">
+    <origin xyz="$(arg robot_origin.x) $(arg robot_origin.y) $(arg robot_origin.z)" rpy="$(arg robot_origin.ax) $(arg robot_origin.ay) $(arg robot_origin.az)"/>
   </xacro:kuka_lwr>
 </robot>

Commit message: fix: remove dots from argument names in urdf files

File: lwr_robot_examples/kuka-lwr-single/lwr_robot/single_lwr_robot/robot/single_lwr_robot.urdf.xacro (robot description, xacro)
@@ -3,13 +3,13 @@
   <xacro:arg name="robot_name" default="lwr"/>
   <xacro:arg name="robot_world" default="world"/>
-  <xacro:arg name="robot_origin.x" default="0"/>
-  <xacro:arg name="robot_origin.y" default="0"/>
-  <xacro:arg name="robot_origin.z" default="0"/>
-  <xacro:arg name="robot_origin.ax" default="0"/>
-  <xacro:arg name="robot_origin.ay" default="0"/>
-  <xacro:arg name="robot_origin.az" default="0"/>  <!-- Include all models -->
+  <xacro:arg name="robot_origin_x" default="0"/>
+  <xacro:arg name="robot_origin_y" default="0"/>
+  <xacro:arg name="robot_origin_z" default="0"/>
+  <xacro:arg name="robot_origin_ax" default="0"/>
+  <xacro:arg name="robot_origin_ay" default="0"/>
+  <xacro:arg name="robot_origin_az" default="0"/>  <!-- Include all models -->
   <xacro:include filename="$(find lwr_description)/model/kuka_lwr.urdf.xacro"/>
   <xacro:kuka_lwr base_link="$(arg robot_world)" name="$(arg robot_name)">
-    <origin xyz="$(arg robot_origin.x) $(arg robot_origin.y) $(arg robot_origin.z)" rpy="$(arg robot_origin.ax) $(arg robot_origin.ay) $(arg robot_origin.az)"/>
+    <origin xyz="$(arg robot_origin_x) $(arg robot_origin_y) $(arg robot_origin_z)" rpy="$(arg robot_origin_ax) $(arg robot_origin_ay) $(arg robot_origin_az)"/>
   </xacro:kuka_lwr>
 </robot>
